File: hardware/automatisch wagentje/Propellor.sch (KiCad schematic (older format))
At the start: 7 parts, among them U1 P8X32A-D40, U3 24LC256, Y1 Crystal

Commit message: test
test
Connections:
- net labels added: IC1.CH_PD, IC1.GPIO0, IC1.GPIO2, IC1.RTS, IC1.RX, IC1.TX
- net labels removed: CH_PD, GPIO0, GPIO2, RTS
- wire segments 41 -> 54
Changed lines of the file:
@@
 Wire Wire Line
 	6495 4010 6645 4010
-Text Label 6635 3910 3    50   ~ 0
+Text Label 6635 3910 2    50   ~ 0
 TX
 Text Label 6645 4010 2    50   ~ 0
@@
 	5095 2510 4975 2510
 Text HLabel 4920 3010 0    50   Input ~ 0
-RX
+IC1.RX
 $Comp
 L MCU_Parallax:P8X32A-D40 U1
@@
 $EndComp
 Text HLabel 4920 2910 0    50   Input ~ 0
-GPIO0
+IC1.GPIO0
 Text HLabel 4915 2810 0    50   Input ~ 0
-RTS
+IC1.RTS
 Text HLabel 4915 2710 0    50   Input ~ 0
-GPIO2
+IC1.GPIO2
 Text HLabel 4910 2610 0    50   Input ~ 0
-CH_PD
+IC1.CH_PD
 Text HLabel 4975 2510 0    50   Input ~ 0
-TX
+IC1.TX
 $Comp
 L programmers:propstick CON?
@@
 	-1   0    0    1
 $EndComp
+Wire Wire Line
+	6495 2510 6800 2510
+Wire Wire Line
+	6495 2610 6805 2610
+Wire Wire Line
+	6495 2710 6805 2710
+Wire Wire Line
+	6495 2810 6810 2810
+Wire Wire Line
+	6495 2910 6815 2910
+Wire Wire Line
+	6495 3010 6820 3010
+Wire Wire Line
+	6495 3110 6830 3110
+Wire Wire Line
+	6495 3210 6830 3210
+Wire Wire Line
+	6495 3310 6840 3310
+Wire Wire Line
+	6495 3410 6840 3410
+Wire Wire Line
+	6495 3510 6845 3510
+Wire Wire Line
+	6495 3710 6685 3710
+Wire Wire Line
+	6495 3810 6680 3810
+Text Label 6680 3810 2    50   ~ 0
+SDA
+Text Label 6685 3710 2    50   ~ 0
+SCL
 $EndSCHEMATC
