File: hardware/automatisch wagentje/MCU.sch (KiCad schematic (older format))
At the start: 5 parts, among them CON1 propstick, U1 P8X32A-D40, U2 24LC256, Y1 Crystal

Commit message: esp82866
esp schema getekend
Parts:
- added C?: 10uf, symbol Device:C
- added C?: 10nF, symbol Device:C
Connections:
- net +3V3: now also C?.1, C?.1
- net GND: now also C?.2, C?.2
Changed lines of the file:
@@
 $Descr A4 11693 8268
 encoding utf-8
-Sheet 2 3
+Sheet 2 4
 Title ""
 Date ""
@@
 NoConn ~ 6450 3570
 NoConn ~ 6450 3670
+$Comp
+L Device:C C?
+U 1 1 5EAD59EE
+P 1575 6140
+F 0 "C?" H 1690 6186 50  0000 L CNN
+F 1 "10uf" H 1690 6095 50  0000 L CNN
+F 2 "" H 1613 5990 50  0001 C CNN
+F 3 "~" H 1575 6140 50  0001 C CNN
+	1    1575 6140
+	1    0    0    -1
+$EndComp
+$Comp
+L ESP32-PoE-ISO_Rev_C:GND #PWR?
+U 1 1 5EAD5FE7
+P 1575 6435
+F 0 "#PWR?" H 1575 6185 50  0001 C CNN
+F 1 "GND" H 1580 6262 50  0000 C CNN
+F 2 "" H 1575 6435 60  0000 C CNN
+F 3 "" H 1575 6435 60  0000 C CNN
+	1    1575 6435
+	1    0    0    -1
+$EndComp
+$Comp
+L power:+3.3V #PWR?
+U 1 1 5EAD8C0E
+P 1575 5845
+F 0 "#PWR?" H 1575 5695 50  0001 C CNN
+F 1 "+3.3V" H 1590 6018 50  0000 C CNN
+F 2 "" H 1575 5845 50  0001 C CNN
+F 3 "" H 1575 5845 50  0001 C CNN
+	1    1575 5845
+	1    0    0    -1
+$EndComp
+Wire Wire Line
+	1575 5990 1575 5845
+Wire Wire Line
+	1575 6435 1575 6290
+$Comp
+L Device:C C?
+U 1 1 5EAE054D
+P 2085 6130
+F 0 "C?" H 2200 6176 50  0000 L CNN
+F 1 "10nF" H 2200 6085 50  0000 L CNN
+F 2 "" H 2123 5980 50  0001 C CNN
+F 3 "~" H 2085 6130 50  0001 C CNN
+	1    2085 6130
+	1    0    0    -1
+$EndComp
+$Comp
+L ESP32-PoE-ISO_Rev_C:GND #PWR?
+U 1 1 5EAE0553
+P 2085 6425
+F 0 "#PWR?" H 2085 6175 50  0001 C CNN
+F 1 "GND" H 2090 6252 50  0000 C CNN
+F 2 "" H 2085 6425 60  0000 C CNN
+F 3 "" H 2085 6425 60  0000 C CNN
+	1    2085 6425
+	1    0    0    -1
+$EndComp
+$Comp
+L power:+3.3V #PWR?
+U 1 1 5EAE0559
+P 2085 5835
+F 0 "#PWR?" H 2085 5685 50  0001 C CNN
+F 1 "+3.3V" H 2100 6008 50  0000 C CNN
+F 2 "" H 2085 5835 50  0001 C CNN
+F 3 "" H 2085 5835 50  0001 C CNN
+	1    2085 5835
+	1    0    0    -1
+$EndComp
+Wire Wire Line
+	2085 5980 2085 5835
+Wire Wire Line
+	2085 6425 2085 6280
 $EndSCHEMATC

Commit message: encoder schema
encoder schema afgemaakt
Parts:
- gave numbers to parts that had none: 2
Changed lines of the file:
@@
 NoConn ~ 6450 3670
 $Comp
-L Device:C C?
+L Device:C C1
 U 1 1 5EAD59EE
 P 1575 6140
-F 0 "C?" H 1690 6186 50  0000 L CNN
+F 0 "C1" H 1690 6186 50  0000 L CNN
 F 1 "10uf" H 1690 6095 50  0000 L CNN
 F 2 "" H 1613 5990 50  0001 C CNN
@@
 $EndComp
 $Comp
-L ESP32-PoE-ISO_Rev_C:GND #PWR?
+L ESP32-PoE-ISO_Rev_C:GND #PWR011
 U 1 1 5EAD5FE7
 P 1575 6435
-F 0 "#PWR?" H 1575 6185 50  0001 C CNN
+F 0 "#PWR011" H 1575 6185 50  0001 C CNN
 F 1 "GND" H 1580 6262 50  0000 C CNN
 F 2 "" H 1575 6435 60  0000 C CNN
@@
 $EndComp
 $Comp
-L power:+3.3V #PWR?
+L power:+3.3V #PWR010
 U 1 1 5EAD8C0E
 P 1575 5845
-F 0 "#PWR?" H 1575 5695 50  0001 C CNN
+F 0 "#PWR010" H 1575 5695 50  0001 C CNN
 F 1 "+3.3V" H 1590 6018 50  0000 C CNN
 F 2 "" H 1575 5845 50  0001 C CNN
@@
 	1575 6435 1575 6290
 $Comp
-L Device:C C?
+L Device:C C2
 U 1 1 5EAE054D
 P 2085 6130
-F 0 "C?" H 2200 6176 50  0000 L CNN
+F 0 "C2" H 2200 6176 50  0000 L CNN
 F 1 "10nF" H 2200 6085 50  0000 L CNN
 F 2 "" H 2123 5980 50  0001 C CNN
@@
 $EndComp
 $Comp
-L ESP32-PoE-ISO_Rev_C:GND #PWR?
+L ESP32-PoE-ISO_Rev_C:GND #PWR013
 U 1 1 5EAE0553
 P 2085 6425
-F 0 "#PWR?" H 2085 6175 50  0001 C CNN
+F 0 "#PWR013" H 2085 6175 50  0001 C CNN
 F 1 "GND" H 2090 6252 50  0000 C CNN
 F 2 "" H 2085 6425 60  0000 C CNN
@@
 $EndComp
 $Comp
-L power:+3.3V #PWR?
+L power:+3.3V #PWR012
 U 1 1 5EAE0559
 P 2085 5835
-F 0 "#PWR?" H 2085 5685 50  0001 C CNN
+F 0 "#PWR012" H 2085 5685 50  0001 C CNN
 F 1 "+3.3V" H 2100 6008 50  0000 C CNN
 F 2 "" H 2085 5835 50  0001 C CNN
