File: hardware/automatisch wagentje/RC.sch (KiCad schematic (older format))
At the start: 3 parts, among them CON2 RC_Connector, CON3 RC_Connector

Commit message: esp82866
esp schema getekend
Parts:
- added C? (x2): 10uf, symbol Device:C
- added C? (x2): 10nF, symbol Device:C
- gave numbers to parts that had none: 1
Connections:
- net +3V3: now also C?.1, C?.1
- net +5V: now also C?.1, C?.1
- net GND: now also C?.2, C?.2, C?.2, C?.2
Changed lines of the file:
@@
 $Descr A4 11693 8268
 encoding utf-8
-Sheet 3 3
+Sheet 3 4
 Title ""
 Date ""
@@
 U 1 1 5EAE14E5
 P 3440 1375
-F 0 "CON?" V 3574 1347 50  0000 R CNN
+F 0 "CON3" V 3574 1347 50  0000 R CNN
 F 1 "RC_Connector" V 3483 1347 50  0000 R CNN
 F 2 "" H 3440 1375 50  0001 C CNN
@@
 U 1 1 5EAE0F7C
 P 2270 1345
-F 0 "CON?" V 2404 1317 50  0000 R CNN
+F 0 "CON2" V 2404 1317 50  0000 R CNN
 F 1 "RC_Connector" V 2313 1317 50  0000 R CNN
 F 2 "" H 2270 1345 50  0001 C CNN
@@
 	2020 1445 2020 1640
 $Comp
-L ESP32-PoE-ISO_Rev_C:GND #PWR?
+L ESP32-PoE-ISO_Rev_C:GND #PWR018
 U 1 1 5EAE279C
 P 2220 1835
-F 0 "#PWR?" H 2220 1585 50  0001 C CNN
+F 0 "#PWR018" H 2220 1585 50  0001 C CNN
 F 1 "GND" H 2225 1662 50  0000 C CNN
 F 2 "" H 2220 1835 60  0000 C CNN
@@
 	2220 1445 2220 1835
 $Comp
-L Jumper:SolderJumper_3_Open JP?
+L Jumper:SolderJumper_3_Open JP1
 U 1 1 5EAE366C
 P 1800 3130
-F 0 "JP?" H 1800 3243 50  0000 C CNN
+F 0 "JP1" H 1800 3243 50  0000 C CNN
 F 1 "SolderJumper_3_Open" H 1800 3334 50  0000 C CNN
 F 2 "" H 1800 3130 50  0001 C CNN
@@
 	1800 2770 2120 2770
 $Comp
-L power:+3.3V #PWR?
+L power:+3.3V #PWR017
 U 1 1 5EAE528A
 P 2145 2995
-F 0 "#PWR?" H 2145 2845 50  0001 C CNN
+F 0 "#PWR017" H 2145 2845 50  0001 C CNN
 F 1 "+3.3V" H 2290 3065 50  0000 C CNN
 F 2 "" H 2145 2995 50  0001 C CNN
@@
 	2145 3130 2145 2995
 $Comp
-L power:+5V #PWR?
+L power:+5V #PWR016
 U 1 1 5EAE681E
 P 1450 2845
-F 0 "#PWR?" H 1450 2695 50  0001 C CNN
+F 0 "#PWR016" H 1450 2695 50  0001 C CNN
 F 1 "+5V" H 1465 3018 50  0000 C CNN
 F 2 "" H 1450 2845 50  0001 C CNN
@@
 	3190 1475 3190 1675
 $Comp
-L ESP32-PoE-ISO_Rev_C:GND #PWR?
+L ESP32-PoE-ISO_Rev_C:GND #PWR019
 U 1 1 5EAEB934
 P 3390 1615
-F 0 "#PWR?" H 3390 1365 50  0001 C CNN
+F 0 "#PWR019" H 3390 1365 50  0001 C CNN
 F 1 "GND" H 3395 1442 50  0000 C CNN
 F 2 "" H 3390 1615 60  0000 C CNN
@@
 Text HLabel 3190 1675 3    50   Input ~ 0
 CON3.RC_OUT
+$Comp
+L Device:C C?
+U 1 1 5EAE411F
+P 1450 5590
+F 0 "C?" H 1565 5636 50  0000 L CNN
+F 1 "10uf" H 1565 5545 50  0000 L CNN
+F 2 "" H 1488 5440 50  0001 C CNN
+F 3 "~" H 1450 5590 50  0001 C CNN
+	1    1450 5590
+	1    0    0    -1
+$EndComp
+$Comp
+L ESP32-PoE-ISO_Rev_C:GND #PWR?
+U 1 1 5EAE4125
+P 1450 5885
+F 0 "#PWR?" H 1450 5635 50  0001 C CNN
+F 1 "GND" H 1455 5712 50  0000 C CNN
+F 2 "" H 1450 5885 60  0000 C CNN
+F 3 "" H 1450 5885 60  0000 C CNN
+	1    1450 5885
+	1    0    0    -1
+$EndComp
+$Comp
+L power:+3.3V #PWR?
+U 1 1 5EAE412B
+P 1450 5295
+F 0 "#PWR?" H 1450 5145 50  0001 C CNN
+F 1 "+3.3V" H 1465 5468 50  0000 C CNN
+F 2 "" H 1450 5295 50  0001 C CNN
+F 3 "" H 1450 5295 50  0001 C CNN
+	1    1450 5295
+	1    0    0    -1
+$EndComp
+Wire Wire Line
+	1450 5440 1450 5295
+Wire Wire Line
+	1450 5885 1450 5740
+$Comp
+L Device:C C?
+U 1 1 5EAE4133
+P 1960 5580
+F 0 "C?" H 2075 5626 50  0000 L CNN
+F 1 "10nF" H 2075 5535 50  0000 L CNN
+F 2 "" H 1998 5430 50  0001 C CNN
+F 3 "~" H 1960 5580 50  0001 C CNN
+	1    1960 5580
+	1    0    0    -1
+$EndComp
+$Comp
+L ESP32-PoE-ISO_Rev_C:GND #PWR?
+U 1 1 5EAE4139
+P 1960 5875
+F 0 "#PWR?" H 1960 5625 50  0001 C CNN
+F 1 "GND" H 1965 5702 50  0000 C CNN
+F 2 "" H 1960 5875 60  0000 C CNN
+F 3 "" H 1960 5875 60  0000 C CNN
+	1    1960 5875
+	1    0    0    -1
+$EndComp
+$Comp
+L power:+3.3V #PWR?
+U 1 1 5EAE413F
+P 1960 5285
+F 0 "#PWR?" H 1960 5135 50  0001 C CNN
+F 1 "+3.3V" H 1975 5458 50  0000 C CNN
+F 2 "" H 1960 5285 50  0001 C CNN
+F 3 "" H 1960 5285 50  0001 C CNN
+	1    1960 5285
+	1    0    0    -1
+$EndComp
+Wire Wire Line
+	1960 5430 1960 5285
+Wire Wire Line
+	1960 5875 1960 5730
+$Comp
+L Device:C C?
+U 1 1 5EAE60A5
+P 2600 5620
+F 0 "C?" H 2715 5666 50  0000 L CNN
+F 1 "10uf" H 2715 5575 50  0000 L CNN
+F 2 "" H 2638 5470 50  0001 C CNN
+F 3 "~" H 2600 5620 50  0001 C CNN
+	1    2600 5620
+	1    0    0    -1
+$EndComp
+$Comp
+L ESP32-PoE-ISO_Rev_C:GND #PWR?
+U 1 1 5EAE60AB
+P 2600 5915
+F 0 "#PWR?" H 2600 5665 50  0001 C CNN
+F 1 "GND" H 2605 5742 50  0000 C CNN
+F 2 "" H 2600 5915 60  0000 C CNN
+F 3 "" H 2600 5915 60  0000 C CNN
+	1    2600 5915
+	1    0    0    -1
+$EndComp
+Wire Wire Line
+	2600 5470 2600 5325
+Wire Wire Line
+	2600 5915 2600 5770
+$Comp
+L Device:C C?
+U 1 1 5EAE60B9
+P 3110 5610
+F 0 "C?" H 3225 5656 50  0000 L CNN
+F 1 "10nF" H 3225 5565 50  0000 L CNN
+F 2 "" H 3148 5460 50  0001 C CNN
+F 3 "~" H 3110 5610 50  0001 C CNN
+	1    3110 5610
+	1    0    0    -1
+$EndComp
+$Comp
+L ESP32-PoE-ISO_Rev_C:GND #PWR?
+U 1 1 5EAE60BF
+P 3110 5905
+F 0 "#PWR?" H 3110 5655 50  0001 C CNN
+F 1 "GND" H 3115 5732 50  0000 C CNN
+F 2 "" H 3110 5905 60  0000 C CNN
+F 3 "" H 3110 5905 60  0000 C CNN
+	1    3110 5905
+	1    0    0    -1
+$EndComp
+Wire Wire Line
+	3110 5460 3110 5315
+Wire Wire Line
+	3110 5905 3110 5760
+$Comp
+L power:+5V #PWR?
+U 1 1 5EAE9901
+P 2600 5325
+F 0 "#PWR?" H 2600 5175 50  0001 C CNN
+F 1 "+5V" H 2615 5498 50  0000 C CNN
+F 2 "" H 2600 5325 50  0001 C CNN
+F 3 "" H 2600 5325 50  0001 C CNN
+	1    2600 5325
+	1    0    0    -1
+$EndComp
+$Comp
+L power:+5V #PWR?
+U 1 1 5EAEA073
+P 3110 5315
+F 0 "#PWR?" H 3110 5165 50  0001 C CNN
+F 1 "+5V" H 3125 5488 50  0000 C CNN
+F 2 "" H 3110 5315 50  0001 C CNN
+F 3 "" H 3110 5315 50  0001 C CNN
+	1    3110 5315
+	1    0    0    -1
+$EndComp
 $EndSCHEMATC

Commit message: encoder schema
encoder schema afgemaakt
Parts:
- added Q1: BSS138DW-7-F, digikey-footprints:SOT-363, symbol dk_Transistors-FETs-MOSFETs-Arrays:BSS138DW-7-F
- added R2, R4, R5: 10K, symbol Device:R
- added R3: R, symbol Device:R
- gave numbers to parts that had none: 4
Connections:
- net +3V3: now also R4.1, R5.1
- net +5V: now also Q1.5 (G1), R2.1, R3.1
- net CON2.RC_OUT: now also Q1.3 (D1), R4.2; no longer CON2.1 (pulse)
- net CON3.RC_OUT: now also Q1.6 (D2), R5.2; no longer CON3.1 (pulse)
- new net RC1: CON2.1 (pulse), Q1.4 (S1), R2.2
- new net RC2: CON3.1 (pulse), R3.2
Other:
- moved on the sheet: CON3
