File: hardware/automatisch wagentje/encoder.sch (KiCad schematic (older format))
At the start: 13 parts

Commit message: encoder schema
encoder schema afgemaakt
Parts:
- added C10, C12: 10nF, symbol Device:C
- added C11, C9: 10uf, symbol Device:C
- gave numbers to parts that had none: 9
Connections:
- net +3V3: now also C10.1, C9.1
- net +5V: now also C11.1, C12.1
- net GND: now also C10.2, C11.2, C12.2, C9.2
- net ENCODER1: now reaches U3.3
- net ENCODER2: now reaches U3.4
- net ENCODER3: now reaches U3.10
- net ENCODER4: now reaches U3.11
