File: hardware/automatisch wagentje/esp.sch (KiCad schematic (older format))
At the start: 3 parts

Commit message: encoder
encoder schema gemaakt
Parts:
- renumbered MOD1 to MOD?
Changed lines of the file:
@@
 $Descr A4 11693 8268
 encoding utf-8
-Sheet 4 4
+Sheet 4 5
 Title ""
 Date ""
@@
 $EndDescr
 $Comp
-L modulles:ESP8266 MOD1
+L modulles:ESP8266 MOD?
 U 1 1 5EACD8E7
 P 5000 3035

Commit message: encoder schema
encoder schema afgemaakt
Parts:
- gave numbers to parts that had none: 3
Changed lines of the file:
@@
 $EndDescr
 $Comp
-L modulles:ESP8266 MOD?
+L modulles:ESP8266 MOD1
 U 1 1 5EACD8E7
 P 5000 3035
-F 0 "MOD?" H 5242 2220 50  0000 C CNN
+F 0 "MOD1" H 5242 2220 50  0000 C CNN
 F 1 "ESP8266" H 5242 2311 50  0000 C CNN
 F 2 "" H 5000 3035 50  0001 C CNN
@@
 AR Path="/5EAD1CB4" Ref="#PWR?"  Part="1"
 AR Path="/5EACD4BB/5EAD1CB4" Ref="#PWR021"  Part="1"
-F 0 "#PWR?" H 5365 2435 50  0001 C CNN
+F 0 "#PWR021" H 5365 2435 50  0001 C CNN
 F 1 "+3.3V" V 5330 2525 50  0000 C CNN
 F 2 "" H 5365 2585 50  0001 C CNN
@@
 AR Path="/5EA957A8/5EAD4136" Ref="#PWR?"  Part="1"
 AR Path="/5EACD4BB/5EAD4136" Ref="#PWR020"  Part="1"
-F 0 "#PWR?" H 5325 2835 50  0001 C CNN
+F 0 "#PWR020" H 5325 2835 50  0001 C CNN
 F 1 "GND" H 5330 2912 50  0000 C CNN
 F 2 "" H 5325 3085 60  0000 C CNN
@@
 MOD1.TX
 $Comp
-L Device:C C?
+L Device:C C7
 U 1 1 5EAEB180
 P 4365 4895
-F 0 "C?" H 4480 4941 50  0000 L CNN
+F 0 "C7" H 4480 4941 50  0000 L CNN
 F 1 "10uf" H 4480 4850 50  0000 L CNN
 F 2 "" H 4403 4745 50  0001 C CNN
@@
 $EndComp
 $Comp
-L ESP32-PoE-ISO_Rev_C:GND #PWR?
+L ESP32-PoE-ISO_Rev_C:GND #PWR035
 U 1 1 5EAEB186
 P 4365 5190
-F 0 "#PWR?" H 4365 4940 50  0001 C CNN
+F 0 "#PWR035" H 4365 4940 50  0001 C CNN
 F 1 "GND" H 4370 5017 50  0000 C CNN
 F 2 "" H 4365 5190 60  0000 C CNN
@@
 $EndComp
 $Comp
-L power:+3.3V #PWR?
+L power:+3.3V #PWR034
 U 1 1 5EAEB18C
 P 4365 4600
-F 0 "#PWR?" H 4365 4450 50  0001 C CNN
+F 0 "#PWR034" H 4365 4450 50  0001 C CNN
 F 1 "+3.3V" H 4380 4773 50  0000 C CNN
 F 2 "" H 4365 4600 50  0001 C CNN
@@
 	4365 5190 4365 5045
 $Comp
-L Device:C C?
+L Device:C C8
 U 1 1 5EAEB194
 P 4875 4885
-F 0 "C?" H 4990 4931 50  0000 L CNN
+F 0 "C8" H 4990 4931 50  0000 L CNN
 F 1 "10nF" H 4990 4840 50  0000 L CNN
 F 2 "" H 4913 4735 50  0001 C CNN
@@
 $EndComp
 $Comp
-L ESP32-PoE-ISO_Rev_C:GND #PWR?
+L ESP32-PoE-ISO_Rev_C:GND #PWR037
 U 1 1 5EAEB19A
 P 4875 5180
-F 0 "#PWR?" H 4875 4930 50  0001 C CNN
+F 0 "#PWR037" H 4875 4930 50  0001 C CNN
 F 1 "GND" H 4880 5007 50  0000 C CNN
 F 2 "" H 4875 5180 60  0000 C CNN
@@
 $EndComp
 $Comp
-L power:+3.3V #PWR?
+L power:+3.3V #PWR036
 U 1 1 5EAEB1A0
 P 4875 4590
-F 0 "#PWR?" H 4875 4440 50  0001 C CNN
+F 0 "#PWR036" H 4875 4440 50  0001 C CNN
 F 1 "+3.3V" H 4890 4763 50  0000 C CNN
 F 2 "" H 4875 4590 50  0001 C CNN
